File: project_files/encoder_debouncing.kicad_sch (KiCad schematic)
At the start: 18 parts, among them J1 Header, J2 Header, SW1 RotaryEncoder_Switch, U1 74HC14

Commit message: values update
Parts:
- C2, C3, C4: value 91nF -> 100nF
Changed lines of the file:
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@@
-(kicad_sch (version 20210621) (generator eeschema)
+(kicad_sch (version 20210406) (generator eeschema)
   (paper "A4")
   (junction (at 86.36 55.88) (diameter 0.9144) (color 0 0 0 0))
@@
       (effects (font (size 1.27 1.27)) (justify left))
     )
-    (property "Value" "91nF" (id 1) (at 120.65 64.1349 0)
+    (property "Value" "100nF" (id 1) (at 120.65 64.1349 0)
       (effects (font (size 1.27 1.27)) (justify left))
     )
@@
       (effects (font (size 1.27 1.27)) (justify left))
     )
-    (property "Value" "91nF" (id 1) (at 120.65 90.8049 0)
+    (property "Value" "100nF" (id 1) (at 120.65 90.8049 0)
       (effects (font (size 1.27 1.27)) (justify left))
     )
@@
       (effects (font (size 1.27 1.27)) (justify left))
     )
-    (property "Value" "91nF" (id 1) (at 120.65 117.4749 0)
+    (property "Value" "100nF" (id 1) (at 120.65 117.4749 0)
       (effects (font (size 1.27 1.27)) (justify left))
     )
@@
     )
     (path "/409b8b1f-818a-4dd3-b7b2-886128876eab"
-      (reference "C2") (unit 1) (value "91nF") (footprint "Capacitor_SMD:C_0603_1608Metric_Pad1.08x0.95mm_HandSolder")
+      (reference "C2") (unit 1) (value "100nF") (footprint "Capacitor_SMD:C_0603_1608Metric_Pad1.08x0.95mm_HandSolder")
     )
     (path "/ac85e57f-5ed5-49e4-8524-cb2e7ae59764"
-      (reference "C3") (unit 1) (value "91nF") (footprint "Capacitor_SMD:C_0603_1608Metric_Pad1.08x0.95mm_HandSolder")
+      (reference "C3") (unit 1) (value "100nF") (footprint "Capacitor_SMD:C_0603_1608Metric_Pad1.08x0.95mm_HandSolder")
     )
     (path "/ab87260f-2bbf-4c41-87cd-28d2bd004a00"
-      (reference "C4") (unit 1) (value "91nF") (footprint "Capacitor_SMD:C_0603_1608Metric_Pad1.08x0.95mm_HandSolder")
+      (reference "C4") (unit 1) (value "100nF") (footprint "Capacitor_SMD:C_0603_1608Metric_Pad1.08x0.95mm_HandSolder")
     )
     (path "/4d5ce7ba-9acb-4515-a748-3227f2abad32"
