File: project_files/0603/encoder_debouncing.kicad_pcb (KiCad board)
At the start: 2 copper layers, 25.4 x 25.4 mm, 18 parts, among them J1 Header, J2 Header, SW1 RotaryEncoder_Switch, U1 74HC14

Commit message: added variation with 0805 components
Parts:
- J1, J2: moved to B.Cu
- SW1: value RotaryEncoder_Switch -> EC11
- turned J1 to 90 degrees
- turned J2 to -90 degrees
Routing:
- net GND: track 41.3 -> 61.6 mm
